File: backplane.sch (KiCad schematic (older format))
At the start: 35 parts, among them J1 I2C, J2 I2C, J3 SER, J4 PWR, J5 PWR, J6 FAN, J7 PPS, Q4 Q_NMOS_GSD, Q5 Q_PMOS_GSD, SW1 SW_Push, U1 Raspberry_Pi_2_3, U2 IC880A-SPI, U3 SHT21, U4 MP1584_MODULE, U5 MCP3425A0T-E/CH

Commit message: modified for base48, different supply, layout
Parts:
- removed C3: C, Capacitors_SMD:C_1206, symbol C
- removed D3: LED_Red, LEDs:LED_1206, symbol LED_Small
- removed D4, D6: D, DO214:DO-214AC, symbol D
- removed F1: Polyfuse, Capacitors_SMD:C_1812, symbol Polyfuse_Small
- removed J2: I2C, headers:header_1x5_unmarked, symbol I2C_HEADER
- removed J3: SER, headers:header_1x2_unmarked, symbol SERIAL_HEADER
- removed J5: PWR, Connectors_Terminal_Blocks:TerminalBlock_Pheonix_MPT-2.54mm_2pol, symbol PWR_HEADER
- removed J6: FAN, headers:header_1x2_marked, symbol FAN
- removed J7: PPS, headers:header_1x1_unmarked, symbol Conn_01x01
- removed Q4: Q_NMOS_GSD, TO_SOT_Packages_SMD:SOT-23, symbol Q_NMOS_GSD
- removed Q5: Q_PMOS_GSD, TO_SOT_Packages_SMD:SOT-23, symbol Q_PMOS_GSD
- removed R10, R11, R12: R, Resistors_SMD:R_0805, symbol R
- removed R13, R9: R, Resistors_SMD:R_1206, symbol R
- removed R3: 220Ω 1/8W, Resistors_SMD:R_1206, symbol R-RESCUE-backplane
- removed SW1: SW_Push, buttons:SW_Mikroshop, symbol SW_Push
- removed U4: MP1584_MODULE, regulators:MP1584_MODULE_ZVEPOWER, symbol MP1584_MODULE
- removed U5: MCP3425A0T-E/CH, TO_SOT_Packages_SMD:SOT-23-6, symbol MCP3425A0T-E/CH-RESCUE-backplane
- added C3: C, Capacitors_SMD:CP_Elec_8x10, symbol device:C
- added D4: D_Schottky, Diodes_SMD:D_SMC, symbol device:D_Schottky
- added D6: D_TVS, Diodes_SMD:D_SMC, symbol device:D_TVS
- added J3: Barrel_Jack, Connectors:BARREL_JACK, symbol Connector:Barrel_Jack
- added J4: GPS_Conn, Socket_Strips:Socket_Strip_Straight_1x05_Pitch2.54mm, symbol Connector:Conn_01x05
- added J5: REG_Conn, Pin_Headers:Pin_Header_Straight_1x03_Pitch2.54mm, symbol Connector:Conn_01x03
- C1: symbol C -> device:C
- C2: footprint capacitor-unmarked:CAP_UNMARKED -> Capacitors_SMD:CP_Elec_8x10; symbol C -> device:C
- D1, D2: footprint LEDs:LED_1206 -> LEDs:LED_0805_HandSoldering; symbol LED_Small -> device:LED_Small
- D5: symbol D_Zener_Small -> device:D_Zener_Small
- J1: footprint headers:header_1x5_unmarked -> Socket_Strips:Socket_Strip_Straight_1x05_Pitch2.54mm; symbol I2C_HEADER -> headers:I2C_HEADER
- J2: renamed from J4; footprint Connectors_Terminal_Blocks:TerminalBlock_Pheonix_MPT-2.54mm_2pol -> TerminalBlock_Phoenix:TerminalBlock_Phoenix_PT-3.5mm_2pol; symbol PWR_HEADER -> headers:PWR_HEADER
- R1, R2: symbol R-RESCUE-backplane -> backplane-rescue:R-RESCUE-backplane
- R4: renamed from R5; symbol R -> device:R
- R5: renamed from R4; symbol R -> device:R
- U1: symbol Raspi_2_3 -> raspi:Raspi_2_3
- U2: symbol IC880A-SPI -> ic880a-spi:IC880A-SPI
- U3: symbol SHT21 -> sensirion:SHT21
Connections:
- net labels added: VIN
- net labels removed: BTN, FAN, GPS_RST, GPS_SUP, LED3
- wire segments 163 -> 122
- no-connect marks 23 -> 30
Other:
- note removed: "A simple button\nconnected to GPIO12.\nIt could be programmed\nto shut down the Rpi\non button press.\n\nNote that you need to\nenable the internal pull-up\nfor the button to work."
- note removed: "ADC"
- note removed: "Button"
- note removed: "Connector for a 5V DC\nfan with a flyback diode."
- note removed: "DC Fan"
- note removed: "The board includes a 5V\npower input/output\nconnector as well as a\nMP1584 step-down\nvoltage regulator for\n6.7-28V input."
- note removed: "This is a 16-Bit\nAnalog-to-Digital\nConverter that is\nwired up to\nmeasure the\nRaspberry Pi\nsupply voltage."
